Commit message: Cambios varios como implementar correctamente los prefix y otras cosas

File: urdf/structures/rbsherkan_chassis/rbsherkan_rocker.urdf.xacro (robot description, xacro)
@@ -1,32 +1,8 @@
 <?xml version="1.0"?>
 <robot name="caster_wheel" xmlns:xacro="http://www.ros.org/wiki/xacro">
-  <xacro:macro name="rocker_front" params="prefix parent *origin hq reflect use_sim:=^|false">
+  <xacro:macro name="rocker_front" params="prefix parent *origin hq reflect">
     <xacro:include filename="$(find robot_description)/urdf/wheels/caster_wheel/rbsherkan_caster.urdf.xacro" />
     <xacro:include filename="$(find robot_description)/urdf/wheels/rubber_wheel/rubber_wheel_150.urdf.xacro" />
     <!-- Base link -->
-    <xacro:if value="${use_sim}">
-    <joint name="${prefix}rocker_joint" type="revolute">
-      <xacro:insert_block name="origin" />
-      <parent link="${parent}"/>
-      <child link="${prefix}rocker_link"/>
-      <axis xyz="0 1 0" />
-      <limit effort="7000.0" lower="-1.0" upper="1.0" velocity="10.0"/>
-      <dynamics damping="0.01" friction="0.1"/>
-    </joint>
-    <transmission name="${prefix}rocker_joint_trans">
-			<type>transmission_interface/SimpleTransmission</type>
-			<joint name="${prefix}rocker_joint">
-				<!-- for the gazebo plugin -->
-				<!--hardwareInterface>EffortJointInterface</hardwareInterface-->
-				<!-- for ros control controller -->
-				<hardwareInterface>hardware_interface/EffortJointInterface</hardwareInterface>
-			</joint>
-			<actuator name="${prefix}rocker_joint_motor">
-				<mechanicalReduction>1</mechanicalReduction>
-				<motorTorqueConstant>20</motorTorqueConstant>
-			</actuator>
-		</transmission>
-  </xacro:if>
-  <xacro:unless value="${use_sim}">
     <joint name="${prefix}rocker_joint" type="fixed">
       <xacro:insert_block name="origin" />
@@ -35,5 +11,4 @@
       <axis xyz="0 1 0" />
     </joint>
-  </xacro:unless>
     <link name="${prefix}rocker_link">
       <visual>
@@ -68,5 +43,5 @@
       </inertial>
     </link>
-    <xacro:rubber_wheel prefix="${prefix}" parent="${prefix}rocker_link" hq="${hq}">
+    <xacro:rubber_wheel prefix="${prefix}wheel_" parent="${prefix}rocker_link" hq="${hq}">
       <xacro:if value="${reflect}">
         <origin xyz="-0.095 0.0579 0.0125" rpy="0 0 0" />
@@ -76,5 +51,5 @@
       </xacro:unless>
     </xacro:rubber_wheel>
-    <xacro:caster prefix="${prefix}caster_" parent="${prefix}rocker_link" hq="${hq}" use_sim="$(arg use_sim)">
+    <xacro:caster prefix="${prefix}caster_" parent="${prefix}rocker_link" hq="${hq}">
       <origin xyz="0.090 0 0.0427" rpy="0 0 0" />
     </xacro:caster>

File: urdf/structures/summit_hm/summit_hm_structure.xacro (robot description, xacro)
@@ -10,4 +10,9 @@
 	  </joint>
 	  <link name="${prefix}_link">
+	    <inertial>
+	      <mass value="0.001"/>
+	      <origin rpy="0 0 0" xyz="0 0 0"/>
+	      <inertia ixx="0.0001" ixy="0" ixz="0" iyy="0.000001" iyz="0" izz="0.0001"/>
+	    </inertial>
 	    <visual>
 	      <origin rpy="0 0 0" xyz="0 0 0"/>
@@ -16,5 +21,5 @@
         </material>
 	      <geometry>
-	        <mesh filename="package://${mesh_file}.dae"/>
+	        <mesh filename="package://${mesh_file}.stl"/>
 	      </geometry>
 	    </visual>

File: urdf/wheels/caster_wheel/rb_theron_caster.urdf.xacro (robot description, xacro)
@@ -10,7 +10,7 @@
   <!-- Caster wheel offset-->
   <xacro:property name="caster_wheel_offset_x" value="-0.033" />
-  <!-- x,y,z in translation from caster_support to the center of the caster wheel-->
   <xacro:property name="caster_wheel_offset_y" value="0.0" />
-  <xacro:property name="caster_wheel_offset_z" value="-0.071" />
+  <xacro:property name="caster_wheel_offset_z" value="-0.08" />
+  <xacro:arg name="use_sim" default="true" />
   <xacro:macro name="cylinder_inertia" params="m r h">
     <inertia  ixx="${m*(3*r*r+h*h)/12}" ixy = "0" ixz = "0"
@@ -18,86 +18,77 @@
               izz="${m*r*r/2}" />
   </xacro:macro>
-  <xacro:macro name="caster" params="prefix parent *origin hq use_sim:=^|false">
-  <!--CASTER SUPPORT -->
-  <xacro:if value="${use_sim}">
-    <joint name="${prefix}joint_support" type="continuous">
-      <parent link="${parent}"/>
-      <child link="${prefix}support"/>
-      <xacro:insert_block name="origin" />
-      <axis xyz="0 0 1" rpy="0 ${M_PI} 0" />
-      <limit effort="100" velocity="100"/>
-      <!-- joint_properties damping="1.5" friction="1.5"/ -->
-      <dynamics damping="0" friction="0.01"/>
-    </joint>
-  </xacro:if>
-  <xacro:unless value="${use_sim}">
-    <joint name="${prefix}joint_support" type="fixed">
+  <xacro:macro name="caster" params="robot_id parent *origin hq use_sim">
+    <!--CASTER SUPPORT -->
+    <xacro:if value="${use_sim}">
+      <joint name="${robot_id}_joint_support" type="continuous">
         <parent link="${parent}"/>
-        <child link="${prefix}support"/>
+        <child link="${robot_id}_support"/>
         <xacro:insert_block name="origin" />
         <axis xyz="0 0 1" rpy="0 ${M_PI} 0" />
-        <!-- <limit effort="100" velocity="100"/> -->
-        <!-- joint_properties damping="1.5" friction="1.5"/ -->
-        <dynamics damping="0" friction="0.01"/>
+        <limit effort="100" velocity="100"/>
+        <dynamics damping="0.8" friction="0.01"/>
       </joint>
-  </xacro:unless>
-    <link name="${prefix}support">
-      <visual>
-        <origin xyz="0 0 0" rpy="0 0 0" />
-          <geometry>
-	       <mesh filename="package://robot_description/meshes/wheels/caster_wheel/caster_wheel.stl" />
-          </geometry>
-      </visual>
-      <collision>
-        <origin xyz="0 0 0" rpy="0 0 0" />
-          <geometry>
-	       <mesh filename="package://robot_description/meshes/wheels/caster_wheel/caster_wheel.dae" />
-          </geometry>
-      </collision>
-      <inertial>
-        <mass value="${caster_support_mass}" />
-        <origin xyz="0 0 0" />
-        <xacro:cylinder_inertia  m="${caster_support_mass}" r="0.010" h="0.010" />  <!--Check these values -->
-      </inertial>
-    </link>
-  <!--CASTER WHEEL -->
-  <!-- xacro:caster_wheel prefix="${prefix}" parent="${prefix}support" hq="${hq}" -->
-  <xacro:caster_wheel prefix="${prefix}" parent="${prefix}support" hq="${hq}" use_sim="$(arg use_sim)">
-		<origin xyz="${caster_wheel_offset_x} ${caster_wheel_offset_y} ${caster_wheel_offset_z}" rpy="0 0 0"/>
-   </xacro:caster_wheel>
- </xacro:macro>
- <xacro:macro name="caster_wheel" params="prefix parent *origin hq use_sim">
+    </xacro:if>
+    <xacro:unless value="${use_sim}">
+      <joint name="${robot_id}_joint_support" type="fixed">
+          <parent link="${parent}"/>
+          <child link="${robot_id}_support"/>
+          <xacro:insert_block name="origin" />
+          <axis xyz="0 0 1" rpy="0 ${M_PI} 0" />
+          <dynamics damping="0" friction="0.01"/>
+        </joint>
+    </xacro:unless>
+      <link name="${robot_id}_support">
+        <visual>
+          <origin xyz="0 0 0" rpy="0 0 0" />
+            <geometry>
+          <mesh filename="package://robot_description/meshes/wheels/caster_wheel/caster_wheel.stl" />
+            </geometry>
+        </visual>
+        <inertial>
+          <mass value="${caster_support_mass}" />
+          <origin xyz="0 0 0" />
+          <xacro:cylinder_inertia  m="${caster_support_mass}" r="0.010" h="0.010" />  <!--Check these values -->
+        </inertial>
+      </link>
+    <!--CASTER WHEEL -->
+    <xacro:caster_wheel robot_id="${robot_id}" parent="${robot_id}_support" hq="${hq}" use_sim="$(arg use_sim)">
+    </xacro:caster_wheel>
+  </xacro:macro>
+ <xacro:macro name="caster_wheel" params="robot_id parent hq use_sim">
   <xacro:if value="${use_sim}">
-    <joint name="${prefix}joint_wheel" type="continuous">
+    <joint name="${robot_id}_joint_wheel" type="continuous">
       <parent link="${parent}"/>
-      <child link="${prefix}wheel"/>
-      <xacro:insert_block name="origin" />
+      <child link="${robot_id}_wheel"/>
+      <origin xyz="-0.033 0.0 -0.071" rpy="0 0 0"/>
       <axis xyz="0 1 0" rpy="0 0 0" />
       <limit effort="100" velocity="100"/>
-      <joint_properties damping="0.1" friction="0.1"/>
+      <joint_properties damping="0.2" friction="2.0"/>
    </joint>
   </xacro:if>
   <xacro:unless value="${use_sim}">
-     <joint name="${prefix}joint_wheel" type="fixed">
+     <joint name="${robot_id}_joint_wheel" type="fixed">
        <parent link="${parent}"/>
-       <child link="${prefix}wheel"/>
-       <xacro:insert_block name="origin" />
+       <child link="${robot_id}_wheel"/>
+      <origin xyz="-0.033 0.0 -0.07" rpy="0 0 0"/>
        <axis xyz="0 1 0" rpy="0 0 0" />
-       <!-- <limit effort="100" velocity="100"/> -->
        <joint_properties damping="0.1" friction="0.1"/>
     </joint>
   </xacro:unless>
-    <link name="${prefix}wheel">
+    <link name="${robot_id}_wheel">
+      <visual>
+          <origin xyz="0 0 0" rpy="${M_PI/2} 0 0" />
+          <geometry>
+            <cylinder length="${caster_height}" radius="${caster_radius}" />
+          </geometry>
+      </visual>
      <collision>
-	  <origin xyz="0 0 0" rpy="${M_PI/2} 0 0" />
-	  <!-- origin xyz="0 0 0" rpy="0 0 0" / -->
-        <geometry>
-		  <!-- mesh filename="package://robot_description/meshes/wheels/mcq_prototype_caster_wheel.dae" / -->
-          <cylinder length="${caster_height}" radius="${caster_radius}" />
-          <!-- sphere radius="${caster_radius}"/ -->
-        </geometry>
-		<surface>
-          <bounce restitution_coefficient = "1"/>
-		</surface>
+        <origin xyz="0 0 0" rpy="${M_PI/2} 0 0" />
+            <geometry>
+              <cylinder length="${caster_height}" radius="${caster_radius}" />
+            </geometry>
+        <surface>
+              <bounce restitution_coefficient = "0.5"/>
+        </surface>
       </collision>
       <inertial>
@@ -109,20 +100,20 @@
   <!-- Transmission is important to link the joints and the controller-->
   <xacro:if value="${use_sim}">
-    <transmission name="${prefix}support_joint_trans">
+    <transmission name="${robot_id}_support_joint_trans">
       <type>transmission_interface/SimpleTransmission</type>
-      <joint name="${prefix}joint_support">
+      <joint name="${robot_id}_joint_support">
           <hardwareInterface>hardware_interface/EffortJointInterface</hardwareInterface>
       </joint>
-      <actuator name="${prefix}support_joint_motor">
+      <actuator name="${robot_id}_support_joint_motor">
         <mechanicalReduction>1</mechanicalReduction>
       	<motorTorqueConstant>1</motorTorqueConstant>
       </actuator>
     </transmission>
-    <transmission name="${prefix}wheel_joint_trans">
+    <transmission name="${robot_id}_wheel_joint_trans">
       <type>transmission_interface/SimpleTransmission</type>
-      <joint name="${prefix}joint_wheel">
+      <joint name="${robot_id}_joint_wheel">
           <hardwareInterface>hardware_interface/EffortJointInterface</hardwareInterface>
       </joint>
-      <actuator name="${prefix}wheel_joint_motor">
+      <actuator name="${robot_id}_wheel_joint_motor">
         <mechanicalReduction>1</mechanicalReduction>
 		<motorTorqueConstant>1</motorTorqueConstant>
@@ -130,5 +121,5 @@
     </transmission>
   </xacro:if>
-    <gazebo reference="${prefix}support">
+    <gazebo reference="${robot_id}_support">
 			<mu1 value="5.0"/>
 			<mu2 value="0.5"/>
@@ -138,5 +129,5 @@
       <turnGravityOff>false</turnGravityOff>
     </gazebo>
-     <gazebo reference="${prefix}wheel">
+     <gazebo reference="${robot_id}_wheel">
 			<mu1 value="100.0"/>
 			<mu2 value="100.0"/>

File: urdf/wheels/caster_wheel/rbsherkan_caster.urdf.xacro (robot description, xacro)
@@ -1,5 +1,5 @@
 <?xml version="1.0"?>
 <robot name="caster" xmlns:xacro="http://www.ros.org/wiki/xacro">
-  <xacro:macro name="caster" params="prefix parent *origin hq use_sim:=^|false">
+  <xacro:macro name="caster" params="prefix parent *origin hq">
     <!-- Caster support parameters -->
     <xacro:property name="caster_support_mass" value="1.5" /> <!-- in kg-->
@@ -18,22 +18,11 @@
     </xacro:macro>
     <!--CASTER SUPPORT -->
-    <xacro:if value="${use_sim}">
-      <joint name="${prefix}support_joint" type="continuous">
-        <xacro:insert_block name="origin" />
-        <parent link="${parent}"/>
-        <child link="${prefix}base_link"/>
-        <axis xyz="0 0 1" />
-        <dynamics damping="0.01" friction="0.1"/>
-      </joint>
-    </xacro:if>
-    <xacro:unless value="${use_sim}">
-      <joint name="${prefix}support_joint" type="fixed">
-        <xacro:insert_block name="origin" />
-        <parent link="${parent}"/>
-        <child link="${prefix}base_link"/>
-        <axis xyz="0 0 1" />
-        <dynamics damping="0.01" friction="0.1"/>
-      </joint>
-    </xacro:unless>
+    <joint name="${prefix}support_joint" type="continuous">
+      <xacro:insert_block name="origin" />
+      <parent link="${parent}"/>
+      <child link="${prefix}base_link"/>
+      <axis xyz="0 0 1" />
+      <dynamics damping="0.01" friction="0.1"/>
+    </joint>
     <link name="${prefix}base_link">
       <visual>
@@ -52,22 +41,11 @@
       </inertial>
     </link>
-    <xacro:if value="${use_sim}">
-      <joint name="${prefix}joint" type="continuous">
-        <origin xyz="${caster_wheel_offset_x} ${caster_wheel_offset_y} ${caster_wheel_offset_z}" rpy="0 0 0" />
-        <parent link="${prefix}base_link"/>
-        <child link="${prefix}link"/>
-        <axis xyz="0 1 0"/>
-        <dynamics damping="0.01" friction="0.1"/>
-      </joint>
-    </xacro:if>
-    <xacro:unless value="${use_sim}">
-      <joint name="${prefix}joint" type="fixed">
-        <origin xyz="${caster_wheel_offset_x} ${caster_wheel_offset_y} ${caster_wheel_offset_z}" rpy="0 0 0" />
-        <parent link="${prefix}base_link"/>
-        <child link="${prefix}link"/>
-        <axis xyz="0 1 0"/>
-        <dynamics damping="0.01" friction="0.1"/>
-      </joint>
-    </xacro:unless>
+    <joint name="${prefix}joint" type="continuous">
+      <origin xyz="${caster_wheel_offset_x} ${caster_wheel_offset_y} ${caster_wheel_offset_z}" rpy="0 0 0" />
+      <parent link="${prefix}base_link"/>
+      <child link="${prefix}link"/>
+      <axis xyz="0 1 0"/>
+      <dynamics damping="0.01" friction="0.1"/>
+    </joint>
     <link name="${prefix}link">
       <!--visual>
@@ -89,27 +67,4 @@
       </inertial>
     </link>
-  <!-- Transmission is important to link the joints and the controller-->
-  <xacro:if value="${use_sim}">
-    <transmission name="${prefix}_support_joint_trans">
-      <type>transmission_interface/SimpleTransmission</type>
-      <joint name="${prefix}support_joint">
-          <hardwareInterface>hardware_interface/EffortJointInterface</hardwareInterface>
-      </joint>
-      <actuator name="${prefix}_support_joint_motor">
-        <mechanicalReduction>1</mechanicalReduction>
-        <motorTorqueConstant>1</motorTorqueConstant>
-      </actuator>
-    </transmission>
-    <transmission name="${prefix}_wheel_joint_trans">
-      <type>transmission_interface/SimpleTransmission</type>
-      <joint name="${prefix}joint">
-          <hardwareInterface>hardware_interface/EffortJointInterface</hardwareInterface>
-      </joint>
-      <actuator name="${prefix}_wheel_joint_motor">
-        <mechanicalReduction>1</mechanicalReduction>
-		<motorTorqueConstant>1</motorTorqueConstant>
-      </actuator>
-    </transmission>
-  </xacro:if>
     <gazebo reference="${prefix}support">
       <mu1>0.45</mu1>

File: urdf/wheels/omni_wheel/rbrobout_omni_wheel.urdf.xacro (robot description, xacro)
@@ -4,6 +4,6 @@
   <!-- Wheels -->
   <xacro:property name="omni_wheel_radius" value="0.127" />
-  <xacro:property name="omni_wheel_height" value="0.128" />
-  <xacro:property name="omni_wheel_mass" value="15" /> <!-- in kg-->
+  <xacro:property name="omni_wheel_height" value="0.087" />
+  <xacro:property name="omni_wheel_mass" value="6.5" /> <!-- in kg-->
   <xacro:macro name="cylinder_inertia" params="m r h">
     <inertia  ixx="${m*(3*r*r+h*h)/12}" ixy = "0" ixz = "0"
@@ -11,17 +11,17 @@
               izz="${m*(3*r*r+h*h)/12}" />
   </xacro:macro>
-  <xacro:macro name="omni_wheel" params="prefix parent *origin reflect hq">
-    <joint name="${prefix}_wheel_joint" type="continuous">
+  <xacro:macro name="rbrobout_omni_wheel" params="prefix1 prefix2 parent *origin reflect hq">
+    <joint name="robot_${prefix2}_wheel_joint" type="continuous">
       <parent link="${parent}"/>
-      <child link="${prefix}_wheel_link"/>
+      <child link="${prefix1}${prefix2}_wheel_link"/>
       <xacro:insert_block name="origin" />
-      <axis xyz="0 0 1" rpy="0 0 0" />
+      <axis xyz="0 1 0" rpy="0 0 0" />
       <limit effort="100" velocity="100"/>
       <joint_properties damping="0.0" friction="0.0"/>
     </joint>
-    <link name="${prefix}_wheel_link">
+    <link name="${prefix1}${prefix2}_wheel_link">
       <visual>
         <xacro:if value="${hq}">
-          <origin xyz="0 0 0" rpy="0 0 0" />
+          <origin xyz="0 0 0" rpy="${PI/2} 0 0" />
           <geometry>
             <mesh filename="package://robot_description/meshes/wheels/omni_wheel/robout_wheel.stl" />
@@ -39,5 +39,5 @@
       </visual>
       <collision>
-				<origin xyz="0 0 0" rpy="0 0 0" />
+				<origin xyz="0 0 0" rpy="${PI/2} 0 0" />
         <geometry>
 					<cylinder length="${omni_wheel_height}" radius="${omni_wheel_radius}" />
@@ -50,21 +50,10 @@
       </inertial>
     </link>
-    <!-- Transmission is important to link the joints and the controller (see summit_xl_control/config/summit_xl_control.yaml)-->
-    <transmission name="${prefix}_wheel_joint_trans">
-      <type>transmission_interface/SimpleTransmission</type>
-      <joint name="${prefix}_wheel_joint" >
-        <hardwareInterface>hardware_interface/VelocityJointInterface</hardwareInterface>
-      </joint>
-      <actuator name="${prefix}_wheel_joint_motor">
-         <mechanicalReduction>1</mechanicalReduction>
-      </actuator>
-    </transmission>
-    <gazebo reference="${prefix}_wheel_link">
-		<mu1 value="0.0"/>
-		<mu2 value="0.0"/>
-		<kp value="10000000.0" />
-		<kd value="1.0" />
-		<fdir1 value="1 0 0"/>
-        <turnGravityOff>false</turnGravityOff>
+    <gazebo reference="${prefix1}${prefix2}_wheel_link">
+      <mu1>0.0</mu1>
+      <mu2>0.0</mu2>
+      <kp>0</kp>
+      <kd>0</kd>
+      <fdir1>0 0 0</fdir1>
     </gazebo>
   </xacro:macro>

File: urdf/wheels/rubber_wheel/gazebo/rubber_wheel.transmission.xacro (robot description, xacro)
@@ -2,9 +2,9 @@
 <robot xmlns:xacro="http://www.ros.org/wiki/xacro">
 	<!-- Rubber wheel transmission -->
-	<xacro:macro name="rubber_wheel_transmission" params="prefix">
+	<xacro:macro name="rubber_wheel_transmission" params="robot_id">
 	<!-- Transmission is important to link the joints and the controller (see rb_theron_control/config/rb_theron_control.yaml)-->
-		<transmission name="${prefix}wheel_joint_trans">
+		<transmission name="${robot_id}_wheel_joint_trans">
 			<type>transmission_interface/SimpleTransmission</type>
-			<joint name="${prefix}wheel_joint">
+			<joint name="${robot_id}_wheel_joint">
 				<!-- for the gazebo plugin -->
 				<!--hardwareInterface>EffortJointInterface</hardwareInterface-->
@@ -12,5 +12,5 @@
 				<hardwareInterface>hardware_interface/VelocityJointInterface</hardwareInterface>
 			</joint>
-			<actuator name="${prefix}wheel_joint_motor">
+			<actuator name="${robot_id}_wheel_joint_motor">
 				<mechanicalReduction>1</mechanicalReduction>
 				<motorTorqueConstant>20</motorTorqueConstant>

File: urdf/wheels/rubber_wheel/rbvogui_rubber_wheel.urdf.xacro (robot description, xacro)
@@ -28,5 +28,10 @@
       <child link="${prefix}wheel"/>
       <xacro:insert_block name="origin" />
-      <axis xyz="0 1 0" rpy="0 0 0" />
+      <xacro:if value="${reflect}">
+        <axis xyz="0 1 0" rpy="0 0 0" />
+      </xacro:if>
+      <xacro:unless value="${reflect}">
+        <axis xyz="0 -1 0" rpy="0 0 0" />
+      </xacro:unless>
       <limit effort="${wheel_joint_effort_limit}" velocity="${wheel_joint_velocity_limit}"/>
       <joint_properties damping="${wheel_joint_damping}" friction="{wheel_joint_friction}"/>

File: urdf/wheels/rubber_wheel/rbvogui_xl_rubber_wheel_285mm.urdf.xacro (robot description, xacro)
@@ -28,5 +28,10 @@
       <child link="${prefix}wheel"/>
       <xacro:insert_block name="origin" />
-      <axis xyz="0 1 0" rpy="0 0 0" />
+      <xacro:if value="${reflect}">
+        <axis xyz="0 -1 0" rpy="0 0 0" />
+      </xacro:if>
+      <xacro:unless value="${reflect}">
+        <axis xyz="0 1 0" rpy="0 0 0" />
+      </xacro:unless>
       <limit effort="${wheel_joint_effort_limit}" velocity="${wheel_joint_velocity_limit}"/>
       <joint_properties damping="${wheel_joint_damping}" friction="{wheel_joint_friction}"/>

File: urdf/wheels/rubber_wheel/rubber_wheel_150.urdf.xacro (robot description, xacro)
@@ -15,9 +15,9 @@
 				  izz="${m*(3*r*r+h*h)/12}" />
 	  </xacro:macro>
-	<xacro:macro name="rubber_wheel" params="prefix parent *origin hq">
+	<xacro:macro name="rubber_wheel" params="robot_id parent *origin hq">
 		<!--WHEEL TIRE -->
-		<joint name="${prefix}wheel_joint" type="continuous">
+		<joint name="${robot_id}_wheel_joint" type="continuous">
 			<parent link="${parent}"/>
-			<child link="${prefix}wheel_link"/>
+			<child link="${robot_id}_wheel_link"/>
 			<xacro:insert_block name="origin" />
 			<axis xyz="0 1 0" rpy="0 0 0" />
@@ -25,5 +25,5 @@
 			<joint_properties damping="0.0" friction="0.0"/>
 		</joint>
-		<link name="${prefix}wheel_link">
+		<link name="${robot_id}_wheel_link">
 			<visual>
 				<!-- HIGH RESOLUTION WHEELS -->
@@ -46,10 +46,10 @@
 			</inertial>
 		</link>
-		<joint name="${prefix}wheel_tire_joint" type="fixed">
-			<parent link="${prefix}wheel_link"/>
-			<child link="${prefix}wheel_tire_link"/>
+		<joint name="${robot_id}_wheel_tire_joint" type="fixed">
+			<parent link="${robot_id}_wheel_link"/>
+			<child link="${robot_id}_wheel_tire_link"/>
 			<origin xyz="0 0 0" rpy="0 0 0" />
 		</joint>
-		<link name="${prefix}wheel_tire_link">
+		<link name="${robot_id}_wheel_tire_link">
 			<visual>
         <origin xyz="0 0 0" rpy="${M_PI/2} 0 0" />
@@ -59,6 +59,6 @@
 			</visual>
 		</link>
-		<xacro:rubber_wheel_transmission prefix="${prefix}" />
-		<xacro:rubber_wheel_gazebo prefix="${prefix}" />
+		<xacro:rubber_wheel_transmission robot_id="${robot_id}" />
+		<xacro:rubber_wheel_gazebo robot_id="${robot_id}" />
 	</xacro:macro>
 </robot>
